File: SI7021-A20-sensor.sch (KiCad schematic (older format))
At the start: 16 parts, among them J1 Conn_01x05, Q1 BSS138, Q2 BSS138, U1 Si7021-A20, U2 MIC5225-3.3

Commit message: update,
Parts:
- D1, D2: footprint LEDs:LED_0805_HandSoldering -> LED_SMD:LED_0805_2012Metric_Pad1.15x1.40mm_HandSolder
- Q1, Q2: footprint TO_SOT_Packages_SMD:SOT-23_Handsoldering -> Package_TO_SOT_SMD:TSOT-23_HandSoldering
- R1, R2, R3, R4, R6: footprint Resistors_SMD:R_0805_HandSoldering -> Resistor_SMD:R_0805_2012Metric_Pad1.15x1.40mm_HandSolder
- R5: footprint w_smd_resistors:r_0805 -> Resistor_SMD:R_0805_2012Metric_Pad1.15x1.40mm_HandSolder
- U1: footprint footprint-lib:DFN-6-1EP_3x3mm_Pitch0.95mm -> w_smd_qfn:dfn6-3x3
- U2: footprint TO_SOT_Packages_SMD:SOT-23-5_HandSoldering -> Package_TO_SOT_SMD:SOT-23-5_HandSoldering
Changed lines of the file:
@@
 F 0 "U1" H 5050 4355 50  0000 C CNN
 F 1 "Si7021-A20" H 5050 4264 50  0000 C CNN
-F 2 "footprint-lib:DFN-6-1EP_3x3mm_Pitch0.95mm" H 5050 3700 50  0001 C CNN
+F 2 "w_smd_qfn:dfn6-3x3" H 5050 3700 50  0001 C CNN
 F 3 "" H 5050 3700 50  0001 C CNN
 F 4 "3x3 6-pin DFN" H 5050 4173 50  0000 C CNN "Field4"
@@
 F 0 "U2" H 8175 4155 50  0000 C CNN
 F 1 "MIC5225-3.3" H 8175 4064 50  0000 C CNN
-F 2 "TO_SOT_Packages_SMD:SOT-23-5_HandSoldering" H 8150 3600 50  0001 C CNN
+F 2 "Package_TO_SOT_SMD:SOT-23-5_HandSoldering" H 8150 3600 50  0001 C CNN
 F 3 "" H 8150 3600 50  0001 C CNN
 F 4 "SOT23-5 " H 8175 3973 50  0000 C CNN "Field4"
@@
 F 0 "Q1" V 5001 1600 50  0000 C CNN
 F 1 "BSS138" V 5092 1600 50  0000 C CNN
-F 2 "TO_SOT_Packages_SMD:SOT-23_Handsoldering" H 4950 1525 50  0001 L CIN
+F 2 "Package_TO_SOT_SMD:TSOT-23_HandSoldering" H 4950 1525 50  0001 L CIN
 F 3 "https://www.fairchildsemi.com/datasheets/BS/BSS138.pdf" H 4750 1600 50  0001 L CNN
 F 4 "SOT-23" V 5183 1600 50  0000 C CNN "Field4"
@@
 F 0 "Q2" V 5600 1950 50  0000 C CNN
 F 1 "BSS138" V 5691 1950 50  0000 C CNN
-F 2 "TO_SOT_Packages_SMD:SOT-23_Handsoldering" H 5550 1875 50  0001 L CIN
+F 2 "Package_TO_SOT_SMD:TSOT-23_HandSoldering" H 5550 1875 50  0001 L CIN
 F 3 "https://www.fairchildsemi.com/datasheets/BS/BSS138.pdf" H 5350 1950 50  0001 L CNN
 F 4 "SOT-23" H 0   0   50  0001 C CNN "Field4"
@@
 F 0 "R1" H 4470 1446 50  0000 L CNN
 F 1 "103" H 4470 1355 50  0000 L CNN
-F 2 "Resistors_SMD:R_0805_HandSoldering" V 4330 1400 50  0001 C CNN
+F 2 "Resistor_SMD:R_0805_2012Metric_Pad1.15x1.40mm_HandSolder" V 4330 1400 50  0001 C CNN
 F 3 "~" H 4400 1400 50  0001 C CNN
 F 4 "0805" H 0   0   50  0001 C CNN "Field4"
@@
 F 0 "R2" H 4470 2346 50  0000 L CNN
 F 1 "103" H 4470 2255 50  0000 L CNN
-F 2 "Resistors_SMD:R_0805_HandSoldering" V 4330 2300 50  0001 C CNN
+F 2 "Resistor_SMD:R_0805_2012Metric_Pad1.15x1.40mm_HandSolder" V 4330 2300 50  0001 C CNN
 F 3 "~" H 4400 2300 50  0001 C CNN
 F 4 "0805" H 0   0   50  0001 C CNN "Field4"
@@
 F 0 "R4" H 5820 2346 50  0000 L CNN
 F 1 "103" H 5820 2255 50  0000 L CNN
-F 2 "Resistors_SMD:R_0805_HandSoldering" V 5680 2300 50  0001 C CNN
+F 2 "Resistor_SMD:R_0805_2012Metric_Pad1.15x1.40mm_HandSolder" V 5680 2300 50  0001 C CNN
 F 3 "~" H 5750 2300 50  0001 C CNN
 F 4 "0805" H 0   0   50  0001 C CNN "Field4"
@@
 F 0 "R3" H 5820 1446 50  0000 L CNN
 F 1 "103" H 5820 1355 50  0000 L CNN
-F 2 "Resistors_SMD:R_0805_HandSoldering" V 5680 1400 50  0001 C CNN
+F 2 "Resistor_SMD:R_0805_2012Metric_Pad1.15x1.40mm_HandSolder" V 5680 1400 50  0001 C CNN
 F 3 "~" H 5750 1400 50  0001 C CNN
 F 4 "0805" H 0   0   50  0001 C CNN "Field4"
@@
 F 0 "R5" H 2020 3546 50  0000 L CNN
 F 1 "102" H 2020 3455 50  0000 L CNN
-F 2 "w_smd_resistors:r_0805" V 1880 3500 50  0001 C CNN
+F 2 "Resistor_SMD:R_0805_2012Metric_Pad1.15x1.40mm_HandSolder" V 1880 3500 50  0001 C CNN
 F 3 "~" H 1950 3500 50  0001 C CNN
 F 4 "0805" H -2450 1200 50  0001 C CNN "Field4"
@@
 F 0 "R6" H 2520 3546 50  0000 L CNN
 F 1 "501" H 2520 3455 50  0000 L CNN
-F 2 "Resistors_SMD:R_0805_HandSoldering" V 2380 3500 50  0001 C CNN
+F 2 "Resistor_SMD:R_0805_2012Metric_Pad1.15x1.40mm_HandSolder" V 2380 3500 50  0001 C CNN
 F 3 "~" H 2450 3500 50  0001 C CNN
 F 4 "0805" H -1950 1200 50  0001 C CNN "Field4"
@@
 F 0 "D1" V 1988 3733 50  0000 R CNN
 F 1 "LED" V 1897 3733 50  0000 R CNN
-F 2 "LEDs:LED_0805_HandSoldering" H 1950 3850 50  0001 C CNN
+F 2 "LED_SMD:LED_0805_2012Metric_Pad1.15x1.40mm_HandSolder" H 1950 3850 50  0001 C CNN
 F 3 "~" H 1950 3850 50  0001 C CNN
 	1    1950 3850
@@
 F 0 "D2" V 2488 3733 50  0000 R CNN
 F 1 "LED" V 2397 3733 50  0000 R CNN
-F 2 "LEDs:LED_0805_HandSoldering" H 2450 3850 50  0001 C CNN
+F 2 "LED_SMD:LED_0805_2012Metric_Pad1.15x1.40mm_HandSolder" H 2450 3850 50  0001 C CNN
 F 3 "~" H 2450 3850 50  0001 C CNN
 	1    2450 3850
