File: SI7021-A20-sensor.kicad_pcb (KiCad board)
At the start: 2 copper layers, 20.1 x 15.7 mm, 16 parts, among them J1 Conn_01x05, Q1 BSS138, Q2 BSS138, U1 Si7021-A20, U2 MIC5225-3.3

Commit message: update,
Parts:
- added REF**: MountingHole_3.2mm_M3, MountingHole:MountingHole_3.2mm_M3, F.Cu at (45.0, 30.0)
- added REF**: MountingHole_3.2mm_M3, MountingHole:MountingHole_3.2mm_M3, F.Cu at (67.0, 30.0)
- added REF**: MountingHole_3.2mm_M3, MountingHole:MountingHole_3.2mm_M3, F.Cu at (45.0, 46.0)
- added REF**: MountingHole_3.2mm_M3, MountingHole:MountingHole_3.2mm_M3, F.Cu at (67.0, 46.0)
- C1, C2, C3: footprint Capacitors_SMD:C_0805_HandSoldering -> Capacitor_SMD:C_0805_2012Metric_Pad1.15x1.40mm_HandSolder
- D1, D2: footprint LEDs:LED_0805_HandSoldering -> LED_SMD:LED_0805_2012Metric_Pad1.15x1.40mm_HandSolder
- J1: footprint footprint-lib:Pin_Header_Straight_1x05_Pitch2.54mm -> footprint-lib.pretty:Pin_Header_Straight_1x05_Pitch2.54mm
- Q1, Q2: footprint TO_SOT_Packages_SMD:SOT-23_Handsoldering -> Package_TO_SOT_SMD:TSOT-23_HandSoldering
- R1, R2, R3, R4, R5, R6: footprint Resistors_SMD:R_0805_HandSoldering -> Resistor_SMD:R_0805_2012Metric_Pad1.15x1.40mm_HandSolder
- U1: footprint footprint-lib:DFN-6-1EP_3x3mm_Pitch0.95mm -> w_smd_qfn:dfn6-3x3
- U2: footprint TO_SOT_Packages_SMD:SOT-23-5_HandSoldering -> Package_TO_SOT_SMD:SOT-23-5_HandSoldering
- moved C1 5.48 mm to (61.1, 39.1)
- moved J1 5.47 mm to (61.0, 43.9)
- moved C3 5.30 mm to (61.1, 36.6)
- moved C2 4.62 mm to (61.1, 33.9)
- moved Q2 4.62 mm to (62.4, 38.0)
- moved R2 4.62 mm to (62.4, 33.8)
- moved D1 4.62 mm to (46.5, 35.4)
- moved D2 4.62 mm to (48.7, 35.4)
- moved Q1 4.62 mm to (52.3, 35.9)
- moved R1 4.62 mm to (52.3, 39.6)
- moved R3 4.62 mm to (52.2, 38.9)
- moved R4 4.62 mm to (54.7, 38.9)
- moved R5 4.62 mm to (46.5, 40.4)
- moved R6 4.62 mm to (48.7, 40.4)
- moved U1 4.62 mm to (57.9, 38.9), turned to 90 degrees
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Connections:
- U2 pad 4: (no net) -> Net-(U2-Pad4)
Routing:
- net /SDA: track 13.6 -> 18.5 mm
- net +5V: track 39.0 -> 42.2 mm
- net +3V3: track 54.0 -> 51.6 mm
- net /SCL: track 12.5 -> 14.4 mm
- net GND: track 45.1 -> 45.6 mm
Other:
- board size 20.1 x 15.7 mm -> 30 x 24 mm
- board text added: "3V3"
- board text added: "GND"
- board text added: "SCL"
- board text added: "SDA"
- board text added: "SI7021-A20"
- board text removed: "SCL SDA +5V +3V3 GND"

Commit message: update
Other:
- board text added: "SI7021-A20 BREAKOUT BOARD"
- board text removed: "SI7021-A20"
Changed lines of the file:
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@@
     (pad 1 np_thru_hole circle (at 0 0) (size 3.2 3.2) (drill 3.2) (layers *.Cu *.Mask))
   )
-  (gr_text SI7021-A20 (at 54.229 27.686) (layer F.SilkS)
-    (effects (font (size 1.2 1.2) (thickness 0.2)))
+  (gr_text "SI7021-A20\nBREAKOUT BOARD" (at 49.53 27.94) (layer F.SilkS)
+    (effects (font (size 1 1) (thickness 0.2)) (justify left))
   )
   (gr_text GND (at 60.96 47.944286 90) (layer F.SilkS)

Commit message: update,
Parts:
- moved C2 2.00 mm to (59.5, 35.0)
- moved C3 1.88 mm to (59.5, 37.5)
- moved C1 1.86 mm to (59.5, 40.0)
- moved R3 1.45 mm to (50.8, 39.0)
- moved R4 1.24 mm to (53.5, 38.9)
Routing:
- net GND: track 45.6 -> 25.3 mm
- net +3V3: track 51.6 -> 48.3 mm
- net +5V: track 42.2 -> 39.8 mm
- net /SDA: track 18.5 -> 16.4 mm

Commit message: update
Routing:
- net GND: vias 1 -> 3
Changed lines of the file:
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@@
     (thickness 1.6)
     (drawings 16)
-    (tracks 115)
+    (tracks 119)
     (zones 0)
     (modules 20)
@@
     (last_trace_width 0.25)
     (trace_clearance 0.2)
-    (zone_clearance 0.4)
+    (zone_clearance 0.3)
     (zone_45_only no)
     (trace_min 0.2)
@@
   (segment (start 57.75 34.105) (end 54.49141 34.105) (width 0.25) (layer F.Cu) (net 1))
   (segment (start 58 34.105) (end 57.75 34.105) (width 0.25) (layer F.Cu) (net 1))
+  (via (at 52.5 41.75) (size 0.8) (drill 0.4) (layers F.Cu B.Cu) (net 1))
+  (via (at 54.9148 39.0144) (size 0.8) (drill 0.4) (layers F.Cu B.Cu) (net 1))
   (segment (start 51.373235 39.769984) (end 51.373235 37.415484) (width 0.25) (layer F.Cu) (net 2) (status 30))
-  (segment (start 56.301 38.931) (end 55.565 38.931) (width 0.25) (layer F.Cu) (net 2) (status 10))
-  (segment (start 55.565 38.931) (end 55.2475 38.6135) (width 0.25) (layer F.Cu) (net 2))
-  (segment (start 55.2475 38.6135) (end 55.2475 37.026) (width 0.25) (layer F.Cu) (net 2))
-  (segment (start 55.3165 36.957) (end 55.2475 37.026) (width 0.25) (layer F.Cu) (net 2))
-  (segment (start 57.023 36.957) (end 55.3165 36.957) (width 0.25) (layer F.Cu) (net 2))
   (segment (start 57.023 36.957) (end 57.531 36.957) (width 0.25) (layer F.Cu) (net 2))
   (segment (start 57.912 36.576) (end 57.912 35.5185) (width 0.25) (layer F.Cu) (net 2) (status 20))
@@
   (segment (start 58.45 43.912) (end 58.42 43.942) (width 0.25) (layer B.Cu) (net 2) (status 30))
   (segment (start 58.45 40.005) (end 58.45 43.912) (width 0.25) (layer B.Cu) (net 2) (status 30))
-  (segment (start 51.25 37.502249) (end 51.373235 37.625484) (width 0.25) (layer F.Cu) (net 2))
-  (segment (start 51.5 32.5) (end 51.25 32.75) (width 0.25) (layer F.Cu) (net 2))
-  (segment (start 54.4715 36.25) (end 54.4715 34.7215) (width 0.25) (layer F.Cu) (net 2))
-  (segment (start 53.5 33.75) (end 53.5 32.75) (width 0.25) (layer F.Cu) (net 2))
-  (segment (start 55.2475 37.026) (end 54.4715 36.25) (width 0.25) (layer F.Cu) (net 2))
-  (segment (start 51.25 32.75) (end 51.25 37.502249) (width 0.25) (layer F.Cu) (net 2))
-  (segment (start 54.4715 34.7215) (end 53.5 33.75) (width 0.25) (layer F.Cu) (net 2))
-  (segment (start 53.25 32.5) (end 51.5 32.5) (width 0.25) (layer F.Cu) (net 2))
-  (segment (start 53.5 32.75) (end 53.25 32.5) (width 0.25) (layer F.Cu) (net 2))
   (segment (start 48.707 41.4) (end 49.85 41.4) (width 0.25) (layer F.Cu) (net 2))
   (segment (start 49.85 41.4) (end 50 41.25) (width 0.25) (layer F.Cu) (net 2))
@@
   (segment (start 58.42 43.942) (end 58.42 41.83) (width 0.25) (layer F.Cu) (net 2))
   (segment (start 58.42 41.83) (end 58.75 41.5) (width 0.25) (layer F.Cu) (net 2))
+  (segment (start 53.5 35) (end 54.25 35.75) (width 0.25) (layer F.Cu) (net 2))
+  (segment (start 51.373235 37.625484) (end 51.25 37.502249) (width 0.25) (layer F.Cu) (net 2))
+  (segment (start 51.25 37.502249) (end 51.25 32.75) (width 0.25) (layer F.Cu) (net 2))
+  (segment (start 51.25 32.75) (end 51.5 32.5) (width 0.25) (layer F.Cu) (net 2))
+  (segment (start 53.5 32.75) (end 53.5 35) (width 0.25) (layer F.Cu) (net 2))
+  (segment (start 51.5 32.5) (end 53.25 32.5) (width 0.25) (layer F.Cu) (net 2))
+  (segment (start 53.25 32.5) (end 53.5 32.75) (width 0.25) (layer F.Cu) (net 2))
+  (segment (start 54.25 35.75) (end 54.25 36.5) (width 0.25) (layer F.Cu) (net 2))
+  (segment (start 54.707 36.957) (end 55.5 36.957) (width 0.25) (layer F.Cu) (net 2))
+  (segment (start 57.023 36.957) (end 55.5 36.957) (width 0.25) (layer F.Cu) (net 2))
+  (segment (start 54.25 36.5) (end 54.707 36.957) (width 0.25) (layer F.Cu) (net 2))
+  (segment (start 55.3165 36.957) (end 55.5 36.957) (width 0.25) (layer F.Cu) (net 2))
+  (segment (start 55.2475 37.026) (end 55.3165 36.957) (width 0.25) (layer F.Cu) (net 2))
+  (segment (start 55.2475 38.4073) (end 55.2475 37.026) (width 0.25) (layer F.Cu) (net 2))
+  (segment (start 56.301 38.931) (end 55.7712 38.931) (width 0.25) (layer F.Cu) (net 2))
+  (segment (start 55.7712 38.931) (end 55.2475 38.4073) (width 0.25) (layer F.Cu) (net 2))
   (via (at 54.7395 33.2795) (size 0.8) (drill 0.4) (layers F.Cu B.Cu) (net 3))
   (segment (start 54.7395 33.2795) (end 54.7395 33.5335) (width 0.25) (layer B.Cu) (net 3))
@@
   (segment (start 48.707 36.7085) (end 48.707 39.025) (width 0.25) (layer F.Cu) (net 9) (status 30))
   (zone (net 1) (net_name GND) (layer F.Cu) (hatch edge 0.508)
-    (connect_pads (clearance 0.4))
+    (connect_pads (clearance 0.3))
     (min_thickness 0.254)
     (fill yes (arc_segments 16) (thermal_gap 0.508) (thermal_bridge_width 0.508))
@@
   )
   (zone (net 1) (net_name GND) (layer B.Cu) (hatch edge 0.508)
-    (connect_pads (clearance 0.4))
+    (connect_pads (clearance 0.3))
     (min_thickness 0.254)
     (fill yes (arc_segments 32) (thermal_gap 0.508) (thermal_bridge_width 0.508))
